Commit message: 20230415 尝试创建多机器人仿真环境，但还没有成功，先备份好的单机器人仿真环境

File: src/vehicle_simulator/urdf/robot.urdf.xacro (robot description, xacro)
@@ -42,5 +42,5 @@
   </link>
   <joint name="lidar_holder_joint" type="fixed">
-    <origin xyz="0.2 0 -0.175" rpy="0 0 0"/>
+    <origin xyz="0.0 0 -0.175" rpy="0 0 0"/>
     <parent link="base_origin"/>
     <child link="lidar_holder"/>
