Commit message: 20230421 修改程序使其可以进行两个机器人的仿真

File: src/vehicle_simulator/urdf/lidar.urdf.xacro (robot description, xacro)
@@ -1,7 +1,15 @@
 <robot xmlns:xacro="http://www.ros.org/wiki/xacro" name="example">
+  <xacro:arg name="gpu" default="false"/>
+  <xacro:property name="gpu" value="$(arg gpu)" />
+  <xacro:arg name="organize_cloud" default="false"/>
+  <xacro:property name="organize_cloud" value="$(arg organize_cloud)" />
   <link name="lidar" />
-  <xacro:include filename="$(find velodyne_description)/urdf/VLP-16.urdf.xacro"/>
+  <!-- <xacro:include filename="$(find velodyne_description)/urdf/VLP-16.urdf.xacro"/>
   <xacro:VLP-16 parent="lidar" name="velodyne" topic="/velodyne_points" hz="5" samples="350" min_range="0.1" organize_cloud="true">
     <origin xyz="0.0 0.0 0" rpy="0 0 0" />
+  </xacro:VLP-16> -->
+  <xacro:include filename="$(find vehicle_simulator)/urdf/VLP-16.urdf.xacro"/>
+  <xacro:VLP-16 parent="lidar" name="velodyne" topic="velodyne_points" organize_cloud="${organize_cloud}" hz="5" samples="350" min_range="0.1" gpu="${gpu}">
+    <origin xyz="0 0 0.0" rpy="0 0 0" />
   </xacro:VLP-16>
 </robot>

File: src/vehicle_simulator/urdf/little_robot.urdf.xacro (robot description, xacro)
@@ -10,6 +10,6 @@
     </gazebo>
   </xacro:macro>
-  <!-- Base Footprint -->
-  <link name="base_footprint" >
+  <!-- Base Origin -->
+  <link name="base_origin" >
     <origin xyz="0 0 0.0" rpy="0 0 0"/>
     <collision>
@@ -21,5 +21,5 @@
   <!-- Base Link -->
   <joint name="footprint" type="fixed" >
-   <parent link="base_footprint" />
+   <parent link="base_origin" />
     <child link="base_link" />
     <origin xyz="0 0 0.3" rpy="0 0 0" />
@@ -38,9 +38,7 @@
     </collision>
     <inertial>
-      <origin xyz="0 0 0"/>
-      <mass value="10"/>
-      <inertia ixx="3.0" ixy="0.0" ixz="0.0"
-               iyy="3.0" iyz="0.0"
-               izz="3.0" />
+      <mass value="1e-5" />
+      <origin xyz="0 0 0" rpy="0 0 0"/>
+      <inertia ixx="1e-6" ixy="0" ixz="0" iyy="1e-6" iyz="0" izz="1e-6" />
     </inertial>
   </link>
@@ -235,6 +233,13 @@
   </gazebo>
   <xacro:gazebo_material ref="camera"  color="Black" />
+  <!-- lidar Link -->
+  <joint name="lidar_joint" type="fixed">
+    <origin xyz="0.0 0 0" rpy="0 0 0"/>
+    <parent link="lidar_holder"/>
+    <child link="lidar"/>
+  </joint>
+  <link name="lidar" />
   <xacro:include filename="$(find vehicle_simulator)/urdf/VLP-16.urdf.xacro"/>
-  <xacro:VLP-16 parent="lidar_holder" name="velodyne" topic="/velodyne_points" organize_cloud="${organize_cloud}" hz="10" samples="440" gpu="${gpu}">
+  <xacro:VLP-16 parent="lidar" name="velodyne" topic="/velodyne_points" organize_cloud="${organize_cloud}" hz="10" samples="440" gpu="${gpu}">
     <origin xyz="0 0 0.35" rpy="0 0 0" />
   </xacro:VLP-16>

Commit message: 20230421 切换到main暂存更改

File: src/vehicle_simulator/urdf/lidar.urdf.xacro (robot description, xacro)
@@ -1,15 +1,7 @@
 <robot xmlns:xacro="http://www.ros.org/wiki/xacro" name="example">
-  <xacro:arg name="gpu" default="false"/>
-  <xacro:property name="gpu" value="$(arg gpu)" />
-  <xacro:arg name="organize_cloud" default="false"/>
-  <xacro:property name="organize_cloud" value="$(arg organize_cloud)" />
   <link name="lidar" />
-  <!-- <xacro:include filename="$(find velodyne_description)/urdf/VLP-16.urdf.xacro"/>
-  <xacro:VLP-16 parent="lidar" name="velodyne" topic="/velodyne_points" hz="5" samples="350" min_range="0.1" organize_cloud="true">
+  <xacro:include filename="$(find velodyne_description)/urdf/VLP-16.urdf.xacro"/>
+  <xacro:VLP-16 parent="lidar" name="velodyne" topic="velodyne_points" hz="5" samples="350" min_range="0.1" organize_cloud="true">
     <origin xyz="0.0 0.0 0" rpy="0 0 0" />
-  </xacro:VLP-16> -->
-  <xacro:include filename="$(find vehicle_simulator)/urdf/VLP-16.urdf.xacro"/>
-  <xacro:VLP-16 parent="lidar" name="velodyne" topic="velodyne_points" organize_cloud="${organize_cloud}" hz="5" samples="350" min_range="0.1" gpu="${gpu}">
-    <origin xyz="0 0 0.0" rpy="0 0 0" />
   </xacro:VLP-16>
 </robot>
