Commit message: 20230421 回退到官方版本，用来搭建仿真环境测试多机算法

File: src/vehicle_simulator/urdf/camera.urdf.xacro (robot description, xacro)
@@ -2,8 +2,7 @@
   <link name="camera">
     <collision>
-      <origin xyz="0.5 0 0" rpy="0 0 0"/>
+      <origin xyz="0 0 0" rpy="0 0 0"/>
       <geometry>
         <box size="0.001 0.001 0.001"/>
-        <!-- <box size="0.1 0.1 0.1"/> -->
       </geometry>
     </collision>

File: src/vehicle_simulator/urdf/lidar.urdf.xacro (robot description, xacro)
@@ -3,5 +3,5 @@
   <xacro:include filename="$(find velodyne_description)/urdf/VLP-16.urdf.xacro"/>
   <xacro:VLP-16 parent="lidar" name="velodyne" topic="/velodyne_points" hz="5" samples="350" min_range="0.1" organize_cloud="true">
-    <origin xyz="0.0 0.0 0" rpy="0 0 0" />
+    <origin xyz="0 0 0" rpy="0 0 0" />
   </xacro:VLP-16>
 </robot>

File: src/vehicle_simulator/urdf/robot.urdf.xacro (robot description, xacro)
@@ -30,5 +30,5 @@
   <link name="lidar_holder">
     <visual>
-      <origin xyz="0.0 0 0" rpy="0 0 0"/>
+      <origin xyz="0 0 0" rpy="0 0 0"/>
       <geometry>
         <cylinder radius="0.03" length="0.35"/>
@@ -42,14 +42,8 @@
   </link>
   <joint name="lidar_holder_joint" type="fixed">
-    <origin xyz="0.2 0 -0.175" rpy="0 0 0"/>
+    <origin xyz="0.0 0 -0.175" rpy="0 0 0"/>
     <parent link="base_origin"/>
     <child link="lidar_holder"/>
   </joint>
-    <!-- lidar
-  <joint name="lidar_joint" type="fixed">                                                                                                                          #设置joint，注意z的值，设为机器人的高度
-      <origin xyz="0 0 0.1" rpy="0 0 0" />
-      <parent link="lidar_holder"/>
-      <child link="velodyne_base_link"/>
-  </joint> -->
   <link name="left_front_wheel">
     <visual>

File: src/velodyne_simulator/velodyne_description/urdf/VLP-16.urdf.xacro (robot description, xacro)
@@ -34,5 +34,5 @@
     </link>
     <joint name="${name}_base_scan_joint" type="fixed" >
-      <origin xyz="0.0 0 0.0377" rpy="0 0 0" />
+      <origin xyz="0 0 0.0377" rpy="0 0 0" />
       <parent link="${name}_base_link" />
       <child link="${name}"/>
